File: arty-scope-expansion-board.kicad_sch (KiCad schematic)
At the start: 20 parts, among them J1 PMOD_A, J2 PMOD_B, J3 PMOD_C, J4 PMOD_D, U1 AD9288, U2 74LS374, U3 74LS374

Commit message: [backup] Recent small changes
Parts:
- JP1: value Jumper_3_Bridged12 -> DFS Select
Other:
- moved on the sheet: C1, C2, C3, C4, C5, C6, C7, C8, J1, J2, J3, J4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

Commit message: [feat] Added part of A channel analog input stage
Rough signal chain, not final:
- BNC (50R)
- overvoltage protection (series R + TVS, 40Vpp)
- fixed pi attenuator -26dB (55.6R / 499R)
- AD8132 as single-ended-to-diff level shifter (DC-coupled, VOCM 2.5V)
- AD8370 VGA (SPI, dual gain range)

TODO: anti-aliasing filter, output driver stage, offset trim DAC
Parts:
- added C10, C11: 1n, Capacitor_SMD:C_0201_0603Metric_Pad0.64x0.40mm_HandSolder, symbol Device:C
- added C9: 100n, Capacitor_SMD:C_0201_0603Metric_Pad0.64x0.40mm_HandSolder, symbol Device:C
- added D1, D2: PTVS5V0Z1USK, Diode_SMD:Nexperia_DSN1608-2_1.6x0.8mm, symbol Diode:PTVS5V0Z1USK
- added J5: Conn_Coaxial, symbol Connector:Conn_Coaxial
- added JP2: Jumper_3_Bridged12, symbol Jumper:Jumper_3_Bridged12
- added R1: 11, symbol Device:R
- added R10: Rt/2, symbol Device:R
- added R11, R12, R3, R7, R8: 499, symbol Device:R
- added R2, R4: 55.6, symbol Device:R
- added R5, R6: 100, symbol Device:R
- added R9: Rt, symbol Device:R
- added U4: AD8370AREZ-RL7, inzynierka.Library:SOP65P640X120-17N, symbol inżynierka:AD8370AREZ-RL7
- added U5: AD8132ARZ, AD8132ARZ:SOIC127P600X175-8N, symbol inżynierka:AD8132ARZ
Connections:
- net +3.3V: now also D2.1 (K)
- net GND: now also C10.1, C11.1, C9.1, D1.2 (A), J5.2 (Ext), JP2.1 (A), R10.1, R2.2, R4.2, U4.10 (OCOM), U4.15 (ICOM), U4.17 (EP), U4.2 (ICOM_2), U4.7 (OCOM_2), U5.6 (V-)
- new net: R11.1, R8.2, U5.1 (-IN)
- new net: R11.2, R5.1, U5.4 (+OUT)
- new net: D1.1 (K), D2.2 (A), R1.1, R2.1, R3.2
- new net: R12.1, R6.1, U5.5 (-OUT)
- new net: R10.2, R8.1
- new net: R12.2, R7.2, U5.8 (+IN)
- new net: JP2.2 (C), R9.1
- new net: J5.1 (In), R1.2
- new net +5VCC: C10.2, C9.2, U4.11 (VCCO), U4.3 (VCCI), U4.4 (PWUP), U4.6 (VCCO_2), U5.3 (V+)
- new net DAC_A: JP2.3 (B)
- new net INHI_A: R5.2, U4.1 (INHI)
- new net INLO_A: R6.2, U4.16 (INLO)
- new net OPHI_A: U4.8 (OPHI)
- new net OPLO_A: U4.9 (OPLO)
- new net PGA_CLK_A: U4.13 (CLCK)
- new net PGA_DATA_A: U4.14 (DATA)
- new net PGA_LATCH_A: U4.12 (LTCH)
- new net SIG_A: R3.1, R4.1, R7.1, R9.2
- new net VOCM_A: C11.2, U4.5 (VOCM), U5.2 (VOCM)
Other:
- moved on the sheet: C1, C2, C3, C4, C5, C6, C7, C8, JP1, U1

Commit message: [feat] Added next part of A channel analog input stage
Some updates:
- driver stage for ADC input A
- correction in input protection stage
- added filtering on VCC of analog stage IC's
Parts:
- removed D1, D2: PTVS5V0Z1USK, Diode_SMD:Nexperia_DSN1608-2_1.6x0.8mm, symbol Diode:PTVS5V0Z1USK
- added C12, C15: 10u, Capacitor_SMD:C_0201_0603Metric_Pad0.64x0.40mm_HandSolder, symbol Device:C
- added C13, C14: 100n, Capacitor_SMD:C_0201_0603Metric_Pad0.64x0.40mm_HandSolder, symbol Device:C
- added C16, C17: 100n, symbol Device:C_Small
- added C18: 47p, Capacitor_SMD:C_0201_0603Metric_Pad0.64x0.40mm_HandSolder, symbol Device:C
- added C19: 10p, Capacitor_SMD:C_0201_0603Metric_Pad0.64x0.40mm_HandSolder, symbol Device:C
- added D3: SD24C-01F, Diode_SMD:D_SOD-323, symbol Diode:SD24C-01F
- added R13: 11, symbol Device:R
- added R15, R16, R17, R18: 499, symbol Device:R
- added R19, R20: 100, symbol Device:R
- added R21: 2.61k, symbol Device:R
- added R22: 10k, symbol Device:R
- added R23, R24: 49.9, symbol Device:R
- added U6: AD8132ARZ, AD8132ARZ:SOIC127P600X175-8N, symbol inżynierka:AD8132ARZ
Connections:
- net +5VCC: now also C12.2, C13.2, C14.2, C15.2, U6.3 (V+)
- net GND: now also C12.1, C13.1, C14.1, C15.1, C16.1, C17.1, D3.2 (A2), R22.1, U6.6 (V-)
- net OPHI_A: now also R15.1
- net OPLO_A: now also R16.1
- net at R2.1, R3.2: now also D3.1 (A1), R13.1; no longer R1.1
- net +AINA: now reaches U1.2 (AINA)
- net +AINA: now also C19.2, R23.2
- net -AINA: now reaches U1.3 (/AINA)
- net -AINA: now also C19.1, R24.2
- net REFOUT: now reaches U1.5 (REFINA)
- net REFOUT: now also U1.6 (REFOUT), U1.7 (REFINB), C16.2, C17.2, R21.2
- new net: R16.2, R18.1, U6.1 (-IN)
- new net: R18.2, R19.1, U6.4 (+OUT)
- new net: R17.1, R20.1, U6.5 (-OUT)
- new net: R15.2, R17.2, U6.8 (+IN)
- new net: C18.2, R19.2, R23.1
- new net: C18.1, R20.2, R24.1
- new net: R1.1, R13.2
- new net REFOUT_VOCM: R21.1, R22.2, U6.2 (VOCM)
Other:
- moved on the sheet: J5, JP1, R1

Commit message: [feat] Added footprints to all A channel elements
TVS diode still doesn't have correct footprint or model. Find one on
LCSC.
Parts:
- added C20: 100n, Capacitor_SMD:C_0201_0603Metric_Pad0.64x0.40mm_HandSolder, symbol Device:C
- added C21: 10u, Capacitor_SMD:C_0201_0603Metric_Pad0.64x0.40mm_HandSolder, symbol Device:C
- added C22, C24: 10u, Capacitor_SMD:C_0603_1608Metric_Pad1.08x0.95mm_HandSolder, symbol Device:C_Small
- added C23, C25: 100n, Capacitor_SMD:C_0603_1608Metric_Pad1.08x0.95mm_HandSolder, symbol Device:C_Small
- added R14, R25, R26: 222, Resistor_SMD:R_2512_6332Metric_Pad1.40x3.35mm_HandSolder, symbol Device:R
- added U7: MCP4822, Package_SO:JEITA_SOIC-8_3.9x4.9mm_P1.27mm, symbol Analog_DAC:MCP4822
- C16, C17: footprint (none) -> Capacitor_SMD:C_0603_1608Metric_Pad1.08x0.95mm_HandSolder
- J5: footprint (none) -> Connector_Coaxial:BNC_TEConnectivity_1478035_Horizontal
- JP2: footprint (none) -> Jumper:SolderJumper-3_P1.3mm_Bridged12_RoundedPad1.0x1.5mm_NumberLabels
- R1, R13, R3, R4: footprint (none) -> Resistor_SMD:R_2512_6332Metric_Pad1.40x3.35mm_HandSolder
- R10, R11, R12, R15, R16, R17, R18, R19, R20, R21, R22, R23, R24, R5, R6, R7, R8, R9: footprint (none) -> Resistor_SMD:R_0201_0603Metric_Pad0.64x0.40mm_HandSolder
- R2: value 55.6 -> 222; footprint (none) -> Resistor_SMD:R_2512_6332Metric_Pad1.40x3.35mm_HandSolder
- U5, U6: footprint AD8132ARZ:SOIC127P600X175-8N -> inzynierka.Library:SOIC127P600X175-8N
Connections:
- net +5VCC: now also C20.2, C21.2, U7.1 (Vdd)
- net DAC_A: now also U7.8 (VA)
- net GND: now also C20.1, C21.1, C22.2, C23.2, C24.2, C25.2, R14.2, R25.2, R26.2, U7.7 (Vss)
- net PGA_CLK_A: now also J1.1 (Pin_1)
- net PGA_DATA_A: now also J1.3 (Pin_3)
- net PGA_LATCH_A: now also J1.5 (Pin_5)
- net VDD: no longer C1.1, C2.1, C3.1, C4.1, C5.1, C6.1, C7.1, C8.1, J1.11 (Pin_11), J1.12 (Pin_12), J2.11 (Pin_11), J2.12 (Pin_12), J3.11 (Pin_11), J3.12 (Pin_12), J4.11 (Pin_11), J4.12 (Pin_12), U1.13 (VD@1), U1.15 (VDD@1), U1.28 (VDD@2), U1.30 (VD@2), U1.31 (VD@3), U1.33 (VDD@3), U1.46 (VDD@4), U1.48 (VD@4)
- net PGA_CLK_B: now reaches J4.1 (Pin_1)
- net PGA_DATA_B: now reaches J4.3 (Pin_3)
- net DAC_CS: now reaches J4.4 (Pin_4)
- net DAC_CS: now also U7.2 (~{CS})
- net PGA_LATCH_B: now reaches J4.5 (Pin_5)
- net DAC_SDI: now reaches J4.6 (Pin_6)
- net DAC_SDI: now also U7.4 (SDI)
- net DAC_LDAC: now reaches J4.7 (Pin_7)
- net DAC_LDAC: now also U7.5 (~{LDAC})
- net DAC_SCK: now reaches J4.8 (Pin_8)
- net DAC_SCK: now also U7.3 (SCK)
- net at D3.1 (A1), R13.1, R2.1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: now also R14.1, R25.1, R26.1
- net +3.3V renamed +3.3VCC
- net +3.3VCC: now also C1.1, C2.1, C3.1, C4.1, C5.1, C6.1, C7.1, C8.1, J1.11 (Pin_11), J1.12 (Pin_12), J2.11 (Pin_11), J2.12 (Pin_12), J3.11 (Pin_11), J3.12 (Pin_12), J4.11 (Pin_11), J4.12 (Pin_12), U1.13 (VD@1), U1.15 (VDD@1), U1.28 (VDD@2), U1.30 (VD@2), U1.31 (VD@3), U1.33 (VDD@3), U1.46 (VDD@4), U1.48 (VD@4), C22.1, C23.1, C24.1, C25.1
- new net DAC_B: U7.6 (VB)
Other:
- moved on the sheet: C1, C12, C13, C16, C17, C2, C3, C4, C5, C6, C7, C8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

Commit message: [feat] Started routing A channel input traces
Input 50 Ohm traces still needs routing. Anty aliasing filter needs
checking if values are correct with some simulation software. Still no
power planes. Serial signals for PGA/VGA and DAC needs logic level
shifters from 3.3V FPGA to 5V signals.
Parts:
- removed JP2: Jumper_3_Bridged12, Jumper:SolderJumper-3_P1.3mm_Bridged12_RoundedPad1.0x1.5mm_NumberLabels, symbol Jumper:Jumper_3_Bridged12
- added C26, C27, C28: 1n, Capacitor_SMD:C_0201_0603Metric_Pad0.64x0.40mm_HandSolder, symbol Device:C
- added JP2: Jumper_2_Bridged, Jumper:SolderJumper-2_P1.3mm_Bridged_RoundedPad1.0x1.5mm, symbol Jumper:Jumper_2_Bridged
- added R27, R28: 20k, Resistor_SMD:R_0201_0603Metric_Pad0.64x0.40mm_HandSolder, symbol Device:R
- R10: value Rt/2 -> 27.8
- R9: value Rt -> 55.6
Connections:
- net +5VCC: no longer U4.11 (VCCO)
- net DAC_A: now also JP2.1 (A), R27.1; no longer U7.8 (VA)
- net DAC_B: now also R28.1; no longer U7.6 (VB)
- net GND: now also R9.1, C26.2, C27.2, C28.1
- net SIG_A: now also JP2.2 (B)
- net AINA-: now reaches U1.10 (/AINB)
- net AINA-: now also C19.1, R24.2
- net AINA+: now reaches U1.11 (AINB)
- net AINA+: now also C19.2, R23.2
- removed net +AINA: C19.2, R23.2, U1.2 (AINA)
- removed net -AINA: C19.1, R24.2, U1.3 (/AINA)
- net OPHI_A renamed OP_A+
- net OPLO_A renamed OP_A-
- new net: C26.1, R27.2, U7.8 (VA)
- new net: C27.1, R28.2, U7.6 (VB)
- new net: C28.2, U4.11 (VCCO)
Other:
- moved on the sheet: C10, R9

Commit message: [feat] Added power planes with LDO's and changed footprints to correct ones
Two power planes where added:
- 3.3V powered by Arty via LDO
- 5V powered via gpio via LDO (can be powered by Arty 5V - i think)
Changed smaller capacitors sizes to correct ones. In prevous iterations
i missmached metric footprints with imperial ones.
Rerouted whole input stage.
Parts:
- added C29, C31: 100n, Capacitor_SMD:C_0603_1608Metric_Pad1.08x0.95mm_HandSolder, symbol Device:C
- added C30, C32: 10u, Capacitor_SMD:C_0603_1608Metric_Pad1.08x0.95mm_HandSolder, symbol Device:C
- added C33: 100n, Capacitor_SMD:C_0603_1608Metric_Pad1.08x0.95mm_HandSolder, symbol Device:C_Small
- added C34, C35, C37: 1u, Capacitor_SMD:C_0805_2012Metric_Pad1.18x1.45mm_HandSolder, symbol Device:C
- added C36: 4u7, Capacitor_SMD:C_0805_2012Metric_Pad1.18x1.45mm_HandSolder, symbol Device:C
- added J6: Conn_01x02_Pin, Connector_PinHeader_2.54mm:PinHeader_1x02_P2.54mm_Vertical, symbol Connector:Conn_01x02_Pin
- added JP3: Jumper_2_Bridged, Jumper:SolderJumper-2_P1.3mm_Bridged_RoundedPad1.0x1.5mm, symbol Jumper:Jumper_2_Bridged
- added U10: MCP1826S, Package_TO_SOT_SMD:SOT-223-3_TabPin2, symbol Regulator_Linear:MCP1826S
- added U11: MIC5504-3.3YM5, Package_TO_SOT_SMD:SOT-23-5, symbol Regulator_Linear:MIC5504-3.3YM5
- added U8, U9: 74AHCT541, Package_SO:SSOP-20_5.3x7.2mm_P0.65mm, symbol 74xx:74AHCT541
- C1, C2, C3, C4, C5, C6, C7, C8: footprint Capacitor_SMD:C_0201_0603Metric_Pad0.64x0.40mm_HandSolder -> Capacitor_SMD:C_0402_1005Metric_Pad0.74x0.62mm_HandSolder
- C10, C11, C12, C13, C14, C15, C18, C19, C28, C9: footprint Capacitor_SMD:C_0201_0603Metric_Pad0.64x0.40mm_HandSolder -> Resistor_SMD:R_0603_1608Metric_Pad0.98x0.95mm_HandSolder
- C16, C17: footprint Capacitor_SMD:C_0603_1608Metric_Pad1.08x0.95mm_HandSolder -> Capacitor_SMD:C_0402_1005Metric_Pad0.74x0.62mm_HandSolder
- C20, C21, C26, C27: footprint Capacitor_SMD:C_0201_0603Metric_Pad0.64x0.40mm_HandSolder -> Capacitor_SMD:C_0603_1608Metric_Pad1.08x0.95mm_HandSolder
- D3: value SD24C-01F -> CDSOD323-T24C
- JP1: footprint Jumper:SolderJumper-3_P1.3mm_Bridged123_RoundedPad1.0x1.5mm_NumberLabels -> Jumper:SolderJumper-3_P1.3mm_Bridged12_RoundedPad1.0x1.5mm_NumberLabels
- R10, R11, R12, R7, R8, R9: footprint Resistor_SMD:R_0201_0603Metric_Pad0.64x0.40mm_HandSolder -> Resistor_SMD:R_0805_2012Metric_Pad1.20x1.40mm_HandSolder
- R15, R16, R17, R18, R19, R20, R21, R22, R23, R24, R27, R28, R5, R6: footprint Resistor_SMD:R_0201_0603Metric_Pad0.64x0.40mm_HandSolder -> Resistor_SMD:R_0603_1608Metric_Pad0.98x0.95mm_HandSolder
Connections:
- net VDD is gone; now on net +3.3VCC: JP1.3 (B)
- net +3.3VCC: now also C33.1, C34.1, U10.3 (VO); no longer J1.11 (Pin_11), J1.12 (Pin_12), J2.11 (Pin_11), J2.12 (Pin_12), J3.11 (Pin_11), J3.12 (Pin_12), J4.11 (Pin_11), J4.12 (Pin_12)
- net +5VCC: now also C29.2, C30.2, C31.2, C32.2, C35.1, U11.5 (VOUT), U8.20 (VCC), U9.20 (VCC)
- net DAC_A: now also R3.1, R4.1, R7.1, R9.2; no longer JP2.1 (A)
- net GND: now also C29.1, C30.1, C31.1, C32.1, C33.2, C34.2, C35.2, C36.2, C37.2, J6.2 (Pin_2), U10.2 (GND), U11.2 (GND), U8.1 (G1), U8.10 (GND), U8.19 (G2), U9.1 (G1), U9.10 (GND), U9.19 (G2)
- net at C26.1, U7.8 (VA): now also JP2.1 (A); no longer R27.2
- net at C27.1, U7.6 (VB): now also JP3.1 (A); no longer R28.2
- net DAC_CS renamed DAC_CS_3.3V
- net DAC_CS_3.3V: now also U9.8 (A6); no longer U7.2 (~{CS})
- net DAC_LDAC renamed DAC_LDAC_3.3V
- net DAC_LDAC_3.3V: now also U9.5 (A3); no longer U7.5 (~{LDAC})
- net DAC_SCK renamed DAC_SCK_3.3V
- net DAC_SCK_3.3V: now also U9.6 (A4); no longer U7.3 (SCK)
- net DAC_SDI renamed DAC_SDI_3.3V
- net DAC_SDI_3.3V: now also U9.7 (A5); no longer U7.4 (SDI)
- net PGA_CLK_A renamed PGA_CLK_A_5V
- net PGA_CLK_A_5V: now also U8.18 (Y0); no longer J1.1 (Pin_1)
- net PGA_CLK_B renamed PGA_CLK_B_3.3V
- net PGA_CLK_B_3.3V: now also U9.2 (A0)
- net PGA_DATA_A renamed PGA_DATA_A_3.3V
- net PGA_DATA_A_3.3V: now also U8.3 (A1); no longer U4.14 (DATA)
- net PGA_DATA_B renamed PGA_DATA_B_3.3V
- net PGA_DATA_B_3.3V: now also U9.3 (A1)
- net PGA_LATCH_A renamed PGA_CLK_A_3.3V
- net PGA_CLK_A_3.3V: now also U8.2 (A0); no longer U4.12 (LTCH)
- net PGA_LATCH_B renamed PGA_LATCH_B_3.3V
- net PGA_LATCH_B_3.3V: now also U9.4 (A2)
- removed net SIG_A: JP2.2 (B), R3.1, R4.1, R7.1, R9.2
- new net: JP2.2 (B), R27.2
- new net: C37.1, J6.1 (Pin_1), U11.1 (VIN), U11.3 (EN)
- new net: JP3.2 (B), R28.2
- new net DAC_CS_5V: U7.2 (~{CS}), U9.12 (Y6)
- new net DAC_LDAC_5V: U7.5 (~{LDAC}), U9.15 (Y3)
- new net DAC_SCK_5V: U7.3 (SCK), U9.14 (Y4)
- new net DAC_SDI_5V: U7.4 (SDI), U9.13 (Y5)
- new net PGA_CLK_B_5V: U9.18 (Y0)
- new net PGA_DATA_A_5V: U4.14 (DATA), U8.17 (Y1)
- new net PGA_DATA_B_5V: U9.17 (Y1)
- new net PGA_LATCH_A_3.3V: J1.1 (Pin_1), U8.4 (A2)
- new net PGA_LATCH_A_5V: U4.12 (LTCH), U8.16 (Y2)
- new net PGA_LATCH_B_5V: U9.16 (Y2)
- new net VIN_3.3V: C36.1, J1.11 (Pin_11), J1.12 (Pin_12), J2.11 (Pin_11), J2.12 (Pin_12), J3.11 (Pin_11), J3.12 (Pin_12), J4.11 (Pin_11), J4.12 (Pin_12), U10.1 (VI)
Other:
- moved on the sheet: C14, C15, C20, C21, C22, C23, C24, C25, C26, C27, C28, J1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

Commit message: [feat] Added second channel with routing
Parts:
- added C38, C41, C46: 100n, Resistor_SMD:R_0603_1608Metric_Pad0.98x0.95mm_HandSolder, symbol Device:C
- added C39, C40, C44: 1n, Resistor_SMD:R_0603_1608Metric_Pad0.98x0.95mm_HandSolder, symbol Device:C
- added C42, C47: 10u, Resistor_SMD:R_0603_1608Metric_Pad0.98x0.95mm_HandSolder, symbol Device:C
- added C43: 47p, Resistor_SMD:R_0603_1608Metric_Pad0.98x0.95mm_HandSolder, symbol Device:C
- added C45: 10p, Resistor_SMD:R_0603_1608Metric_Pad0.98x0.95mm_HandSolder, symbol Device:C
- added D4: CDSOD323-T24C, Diode_SMD:D_SOD-323, symbol Diode:SD24C-01F
- added J7: Conn_Coaxial, Connector_Coaxial:BNC_TEConnectivity_1478035_Horizontal, symbol Connector:Conn_Coaxial
- added R29, R30, R32, R33: 499, Resistor_SMD:R_0603_1608Metric_Pad0.98x0.95mm_HandSolder, symbol Device:R
- added R31, R34: 11, Resistor_SMD:R_2512_6332Metric_Pad1.40x3.35mm_HandSolder, symbol Device:R
- added R35, R36, R37, R38: 222, Resistor_SMD:R_2512_6332Metric_Pad1.40x3.35mm_HandSolder, symbol Device:R
- added R39: 499, Resistor_SMD:R_2512_6332Metric_Pad1.40x3.35mm_HandSolder, symbol Device:R
- added R40: 55.6, Resistor_SMD:R_2512_6332Metric_Pad1.40x3.35mm_HandSolder, symbol Device:R
- added R41, R42, R53, R54: 100, Resistor_SMD:R_0603_1608Metric_Pad0.98x0.95mm_HandSolder, symbol Device:R
- added R43, R44: 49.9, Resistor_SMD:R_0603_1608Metric_Pad0.98x0.95mm_HandSolder, symbol Device:R
- added R45: 2.61k, Resistor_SMD:R_0603_1608Metric_Pad0.98x0.95mm_HandSolder, symbol Device:R
- added R46: 10k, Resistor_SMD:R_0603_1608Metric_Pad0.98x0.95mm_HandSolder, symbol Device:R
- added R47: 55.6, Resistor_SMD:R_0805_2012Metric_Pad1.20x1.40mm_HandSolder, symbol Device:R
- added R48: 27.8, Resistor_SMD:R_0805_2012Metric_Pad1.20x1.40mm_HandSolder, symbol Device:R
- added R49, R50, R51, R52: 499, Resistor_SMD:R_0805_2012Metric_Pad1.20x1.40mm_HandSolder, symbol Device:R
- added U12, U14: AD8132ARZ, inzynierka.Library:SOIC127P600X175-8N, symbol inżynierka:AD8132ARZ
- added U13: AD8370AREZ-RL7, inzynierka.Library:SOP65P640X120-17N, symbol inżynierka:AD8370AREZ-RL7
Connections:
- net +5VCC: now also C38.2, C39.2, C41.2, C42.2, C46.2, C47.2, U12.3 (V+), U13.3 (VCCI), U13.4 (PWUP), U13.6 (VCCO_2), U14.3 (V+)
- net DAC_B: now also R39.1, R40.1, R47.2, R49.1
- net GND: now also C38.1, C39.1, C40.1, C41.1, C42.1, C44.1, C46.1, C47.1, D4.2 (A2), J7.2 (Ext), R35.2, R36.2, R37.2, R38.2, R40.2, R46.1, R47.1, R48.1, U12.6 (V-), U13.10 (OCOM), U13.15 (ICOM), U13.17 (EP), U13.2 (ICOM_2), U13.7 (OCOM_2), U14.6 (V-)
- net PGA_CLK_B_5V: now also U13.13 (CLCK)
- net PGA_DATA_B_5V: now also U13.14 (DATA)
- net PGA_LATCH_B_5V: now also U13.12 (LTCH)
- net REFOUT: now also R45.2
- net REFOUT_VOCM: now also R45.1, R46.2, U12.2 (VOCM)
- net AINB+: now reaches U1.2 (AINA)
- net AINB+: now also C45.2, R43.2
- net AINB-: now reaches U1.3 (/AINA)
- net AINB-: now also C45.1, R44.2
- new net: J7.1 (In), R31.2
- new net: R49.2, R51.2, U14.8 (+IN)
- new net: C43.2, R41.2, R43.1
- new net: R30.2, R33.1, U12.1 (-IN)
- new net: R33.2, R41.1, U12.4 (+OUT)
- new net: R32.1, R42.1, U12.5 (-OUT)
- new net: R29.2, R32.2, U12.8 (+IN)
- new net: C40.2, U13.11 (VCCO)
- new net: R51.1, R54.1, U14.5 (-OUT)
- new net: D4.1 (A1), R34.1, R35.1, R36.1, R37.1, R38.1, R39.2
- new net: R31.1, R34.2
- new net: C43.1, R42.2, R44.1
- new net: R50.2, R52.1, U14.1 (-IN)
- new net: R52.2, R53.1, U14.4 (+OUT)
- new net: R48.2, R50.1
- new net INHI_B: R53.2, U13.1 (INHI)
- new net INLO_B: R54.2, U13.16 (INLO)
- new net OP_B+: R29.1, U13.8 (OPHI)
- new net OP_B-: R30.1, U13.9 (OPLO)
- new net VOCM_B: C44.2, U13.5 (VOCM), U14.2 (VOCM)
Other:
- note added: "Channel A"
- note added: "Channel B"

Commit message: [feat] Changed input stage routing, corrected DRC errors, added some silk labels
Parts:
- removed C10, C11, C28, C39, C40, C44: 1n, Resistor_SMD:R_0603_1608Metric_Pad0.98x0.95mm_HandSolder, symbol Device:C
- removed C12, C15, C42, C47: 10u, Resistor_SMD:R_0603_1608Metric_Pad0.98x0.95mm_HandSolder, symbol Device:C
- removed C13, C14, C38, C41, C46, C9: 100n, Resistor_SMD:R_0603_1608Metric_Pad0.98x0.95mm_HandSolder, symbol Device:C
- removed C18, C43: 47p, Resistor_SMD:R_0603_1608Metric_Pad0.98x0.95mm_HandSolder, symbol Device:C
- removed C19, C45: 10p, Resistor_SMD:R_0603_1608Metric_Pad0.98x0.95mm_HandSolder, symbol Device:C
- removed D3, D4: CDSOD323-T24C, Diode_SMD:D_SOD-323, symbol Diode:SD24C-01F
- removed J5, J7: Conn_Coaxial, Connector_Coaxial:BNC_TEConnectivity_1478035_Horizontal, symbol Connector:Conn_Coaxial
- removed R1, R13, R31, R34: 11, Resistor_SMD:R_2512_6332Metric_Pad1.40x3.35mm_HandSolder, symbol Device:R
- removed R10, R48: 27.8, Resistor_SMD:R_0805_2012Metric_Pad1.20x1.40mm_HandSolder, symbol Device:R
- removed R11, R12, R49, R50, R51, R52, R7, R8: 499, Resistor_SMD:R_0805_2012Metric_Pad1.20x1.40mm_HandSolder, symbol Device:R
- removed R14, R2, R25, R26, R35, R36, R37, R38: 222, Resistor_SMD:R_2512_6332Metric_Pad1.40x3.35mm_HandSolder, symbol Device:R
- removed R15, R16, R17, R18, R29, R30, R32, R33: 499, Resistor_SMD:R_0603_1608Metric_Pad0.98x0.95mm_HandSolder, symbol Device:R
- removed R19, R20, R41, R42, R5, R53, R54, R6: 100, Resistor_SMD:R_0603_1608Metric_Pad0.98x0.95mm_HandSolder, symbol Device:R
- removed R21, R45: 2.61k, Resistor_SMD:R_0603_1608Metric_Pad0.98x0.95mm_HandSolder, symbol Device:R
- removed R22, R46: 10k, Resistor_SMD:R_0603_1608Metric_Pad0.98x0.95mm_HandSolder, symbol Device:R
- removed R23, R24, R43, R44: 49.9, Resistor_SMD:R_0603_1608Metric_Pad0.98x0.95mm_HandSolder, symbol Device:R
- removed R3, R39: 499, Resistor_SMD:R_2512_6332Metric_Pad1.40x3.35mm_HandSolder, symbol Device:R
- removed R4, R40: 55.6, Resistor_SMD:R_2512_6332Metric_Pad1.40x3.35mm_HandSolder, symbol Device:R
- removed R47, R9: 55.6, Resistor_SMD:R_0805_2012Metric_Pad1.20x1.40mm_HandSolder, symbol Device:R
- removed U12, U14, U5, U6: AD8132ARZ, inzynierka.Library:SOIC127P600X175-8N, symbol inżynierka:AD8132ARZ
- removed U13, U4: AD8370AREZ-RL7, inzynierka.Library:SOP65P640X120-17N, symbol inżynierka:AD8370AREZ-RL7
Connections:
- net VIN_3.3V: no longer J1.11 (Pin_11), J1.12 (Pin_12), J2.11 (Pin_11), J2.12 (Pin_12), J4.11 (Pin_11), J4.12 (Pin_12)
Other:
- note added: "ADC"
- note removed: "Channel A"
- note removed: "Channel B"
- moved on the sheet: C1, C16, C17, C2, C20, C21, C22, C23, C24, C25, C26, C27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
