File: digital.kicad_sch (KiCad schematic)
At the start: 0 parts

Commit message: [feat] Changed input stage routing, corrected DRC errors, added some silk labels
Parts:
- added C10, C11, C28, C39, C40, C44: 1n, Resistor_SMD:R_0603_1608Metric_Pad0.98x0.95mm_HandSolder, symbol Device:C
- added C12, C15, C42, C47: 10u, Resistor_SMD:R_0603_1608Metric_Pad0.98x0.95mm_HandSolder, symbol Device:C
- added C13, C14, C38, C41, C46, C9: 100n, Resistor_SMD:R_0603_1608Metric_Pad0.98x0.95mm_HandSolder, symbol Device:C
- added C18, C43: 47p, Resistor_SMD:R_0603_1608Metric_Pad0.98x0.95mm_HandSolder, symbol Device:C
- added C19, C45: 10p, Resistor_SMD:R_0603_1608Metric_Pad0.98x0.95mm_HandSolder, symbol Device:C
- added D3, D4: CDSOD323-T24C, Diode_SMD:D_SOD-323, symbol Diode:SD24C-01F
- added J5, J7: Conn_Coaxial, Connector_Coaxial:BNC_TEConnectivity_1478035_Horizontal, symbol Connector:Conn_Coaxial
- added R1, R13, R31, R34: 11, Resistor_SMD:R_2512_6332Metric_Pad1.40x3.35mm_HandSolder, symbol Device:R
- added R10, R48: 27.8, Resistor_SMD:R_0805_2012Metric_Pad1.20x1.40mm_HandSolder, symbol Device:R
- added R11, R12, R49, R50, R51, R52, R7, R8: 499, Resistor_SMD:R_0805_2012Metric_Pad1.20x1.40mm_HandSolder, symbol Device:R
- added R14, R2, R25, R26, R35, R36, R37, R38: 222, Resistor_SMD:R_2512_6332Metric_Pad1.40x3.35mm_HandSolder, symbol Device:R
- added R15, R16, R17, R18, R29, R30, R32, R33: 499, Resistor_SMD:R_0603_1608Metric_Pad0.98x0.95mm_HandSolder, symbol Device:R
- added R19, R20, R41, R42, R5, R53, R54, R6: 100, Resistor_SMD:R_0603_1608Metric_Pad0.98x0.95mm_HandSolder, symbol Device:R
- added R21, R45: 2.61k, Resistor_SMD:R_0603_1608Metric_Pad0.98x0.95mm_HandSolder, symbol Device:R
- added R22, R46: 10k, Resistor_SMD:R_0603_1608Metric_Pad0.98x0.95mm_HandSolder, symbol Device:R
- added R23, R24, R43, R44: 49.9, Resistor_SMD:R_0603_1608Metric_Pad0.98x0.95mm_HandSolder, symbol Device:R
- added R3, R39: 499, Resistor_SMD:R_2512_6332Metric_Pad1.40x3.35mm_HandSolder, symbol Device:R
- added R4, R40: 55.6, Resistor_SMD:R_2512_6332Metric_Pad1.40x3.35mm_HandSolder, symbol Device:R
- added R47, R9: 55.6, Resistor_SMD:R_0805_2012Metric_Pad1.20x1.40mm_HandSolder, symbol Device:R
- added U12, U14, U5, U6: AD8132ARZ, inzynierka.Library:SOIC127P600X175-8N, symbol inżynierka:AD8132ARZ
- added U13, U4: AD8370AREZ-RL7, inzynierka.Library:SOP65P640X120-17N, symbol inżynierka:AD8370AREZ-RL7
Connections:
- new net: R49.2, R51.2, U14.8 (+IN)
- new net: R10.2, R8.1
- new net: R11.1, R8.2, U5.1 (-IN)
- new net: R11.2, R5.1, U5.4 (+OUT)
- new net: R12.1, R6.1, U5.5 (-OUT)
- new net: R12.2, R7.2, U5.8 (+IN)
- new net: D3.1 (A1), R13.1, R14.1, R2.1, R25.1, R26.1, R3.2
- new net: J7.1 (In), R31.2
- new net: R48.2, R50.1
- new net: R50.2, R52.1, U14.1 (-IN)
- new net: C18.2, R19.2, R23.1
- new net: C40.2, U13.11 (VCCO)
- new net: R16.2, R18.1, U6.1 (-IN)
- new net: R18.2, R19.1, U6.4 (+OUT)
- new net: R30.2, R33.1, U12.1 (-IN)
- new net: D4.1 (A1), R34.1, R35.1, R36.1, R37.1, R38.1, R39.2
- new net: R32.1, R42.1, U12.5 (-OUT)
- new net: C43.1, R42.2, R44.1
- new net: C43.2, R41.2, R43.1
- new net: R15.2, R17.2, U6.8 (+IN)
- new net: R52.2, R53.1, U14.4 (+OUT)
- new net: C18.1, R20.2, R24.1
- new net: R51.1, R54.1, U14.5 (-OUT)
- new net: C28.2, U4.11 (VCCO)
- new net: R31.1, R34.2
- new net: R29.2, R32.2, U12.8 (+IN)
- new net: J5.1 (In), R1.2
- new net: R17.1, R20.1, U6.5 (-OUT)
- new net: R33.2, R41.1, U12.4 (+OUT)
- new net: R1.1, R13.2
- new net +5VCC: C10.2, C12.2, C13.2, C14.2, C15.2, C38.2, C39.2, C41.2, C42.2, C46.2, C47.2, C9.2, U12.3 (V+), U13.3 (VCCI), U13.4 (PWUP), U13.6 (VCCO_2), U14.3 (V+), U4.3 (VCCI), U4.4 (PWUP), U4.6 (VCCO_2), U5.3 (V+), U6.3 (V+)
- new net AINA+: C19.2, R23.2
- new net AINA-: C19.1, R24.2
- new net AINB+: C45.2, R43.2
- new net AINB-: C45.1, R44.2
- new net DAC_A: R3.1, R4.1, R7.1, R9.2
- new net DAC_B: R39.1, R40.1, R47.2, R49.1
- new net GND: C10.1, C11.1, C12.1, C13.1, C14.1, C15.1, C28.1, C38.1, C39.1, C40.1, C41.1, C42.1, C44.1, C46.1, C47.1, C9.1, D3.2 (A2), D4.2 (A2), J5.2 (Ext), J7.2 (Ext), R10.1, R14.2, R2.2, R22.1, R25.2, R26.2, R35.2, R36.2, R37.2, R38.2, R4.2, R40.2, R46.1, R47.1, R48.1, R9.1, U12.6 (V-), U13.10 (OCOM), U13.15 (ICOM), U13.17 (EP), U13.2 (ICOM_2), U13.7 (OCOM_2), U14.6 (V-), U4.10 (OCOM), U4.15 (ICOM), U4.17 (EP), U4.2 (ICOM_2), U4.7 (OCOM_2), U5.6 (V-), U6.6 (V-)
- new net INHI_A: R5.2, U4.1 (INHI)
- new net INHI_B: R53.2, U13.1 (INHI)
- new net INLO_A: R6.2, U4.16 (INLO)
- new net INLO_B: R54.2, U13.16 (INLO)
- new net OP_A+: R15.1, U4.8 (OPHI)
- new net OP_A-: R16.1, U4.9 (OPLO)
- new net OP_B+: R29.1, U13.8 (OPHI)
- new net OP_B-: R30.1, U13.9 (OPLO)
- new net PGA_CLK_A_5V: U4.13 (CLCK)
- new net PGA_CLK_B_5V: U13.13 (CLCK)
- new net PGA_DATA_A_5V: U4.14 (DATA)
- new net PGA_DATA_B_5V: U13.14 (DATA)
- new net PGA_LATCH_A_5V: U4.12 (LTCH)
- new net PGA_LATCH_B_5V: U13.12 (LTCH)
- new net REFOUT: R21.2, R45.2
- new net REFOUT_VOCM_A: R21.1, R22.2, U6.2 (VOCM)
- new net REFOUT_VOCM_B: R45.1, R46.2, U12.2 (VOCM)
- new net VOCM_A: C11.2, U4.5 (VOCM), U5.2 (VOCM)
- new net VOCM_B: C44.2, U13.5 (VOCM), U14.2 (VOCM)
Other:
- note added: "Channel A"
- note added: "Channel B"

Commit message: [backup] ---
Parts:
- J5: footprint Connector_Coaxial:BNC_TEConnectivity_1478035_Horizontal -> Connector_Coaxial:BNC_TEConnectivity_1478204_Vertical
Changed lines of the file:
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@@
 		(dnp no)
 		(property "Reference" "D3"
-			(at 61.214 84.582 90)
+			(at 69.85 83.058 90)
 			(show_name no)
 			(do_not_autoplace no)
@@
 		(property "Value" "CDSOD323-T24C"
 			(at 61.214 87.122 90)
+			(hide yes)
 			(show_name no)
 			(do_not_autoplace no)
@@
 			)
 		)
-		(property "Footprint" "Connector_Coaxial:BNC_TEConnectivity_1478035_Horizontal"
+		(property "Footprint" "Connector_Coaxial:BNC_TEConnectivity_1478204_Vertical"
 			(at 44.45 78.74 0)
 			(hide yes)
